Commit message: add costmap

File: src/simulation/chicken_simulator/urdf/kokko.urdf (robot description, URDF)
Before this commit: robot chicken, 7 links, 6 joints
Links:
- removed link hokuyo_link
- added link laser_frame, mass 1e-5; collision box size=0.1 0.1 0.1; visual box size=0.1 0.1 0.1
Joints:
- removed joint hokuyo_joint
- added joint laser_frame_joint: type fixed, parent base_link, child laser_frame, origin xyz=0.1 0 0.15 rpy=0 0 0, axis 0 1 0
